File: kicad_files/solarOSE_kicad.kicad_pcb (KiCad board)
At the start: 2 copper layers, 270.5 x 115.6 mm, 49 parts, among them J1 Conn_01x02, J2 Conn_01x02, J3 Conn_01x02, U1 MCP23017_SP, U2 MCP23017_SP, U3 MCP23017_SP, U4 MCP23017_SP

Commit message: version with one card for 5 motors
Parts:
- removed A10, A11, A12, A13, A14, A15, A16, A17, A18, A19, A20, A6, A7, A8, A9: Pololu_Breakout_A4988, Module:Pololu_Breakout-16_15.2x20.3mm
- removed JM10, JM11, JM12, JM13, JM14, JM15, JM16, JM17, JM18, JM19, JM20, JM6, JM7, JM8, JM9: Conn_01x04_Male, Connector_Wire:SolderWirePad_1x04_P6.35mm_Drill2mm
- removed U2, U3, U4: MCP23017_SP, Package_DIP:DIP-28_W7.62mm
- added J4: Conn_01x03, Connector_Wire:SolderWirePad_1x03_P3.81mm_Drill1.2mm, F.Cu at (142.2, 87.6)
- added J5: Conn_01x03, Connector_Wire:SolderWirePad_1x03_P3.81mm_Drill1.2mm, F.Cu at (142.2, 82.5)
- added J6: Conn_01x03, Connector_Wire:SolderWirePad_1x03_P3.81mm_Drill1.2mm, F.Cu at (142.2, 76.2)
- moved J3 144.0 mm to (92.7, 82.5), turned to 90 degrees
- moved C2 84.1 mm to (180.3, 81.3)
- moved J1 73.7 mm to (162.6, 83.8), turned to 270 degrees
- moved U1 73.3 mm to (132.1, 77.5)
- moved J2 72.0 mm to (205.7, 81.3), turned to 270 degrees
- moved A5 71.2 mm to (199.4, 52.1)
- moved JM5 71.1 mm to (195.6, 43.2)
- moved JM4 69.9 mm to (167.6, 43.2)
- moved A3 68.7 mm to (143.5, 52.1)
- moved A4 68.7 mm to (171.4, 52.1)
- moved JM3 68.6 mm to (139.7, 43.2)
- moved A2 67.4 mm to (115.6, 52.1)
- moved JM2 67.0 mm to (111.4, 43.2)
- moved JM1 66.1 mm to (83.8, 43.2)
- moved A1 64.9 mm to (87.6, 52.1)
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Connections:
- C1 pad 1: GND -> +36V
- C1 pad 2: +36V -> GND
- C2 pad 1: GND -> +36V
- C2 pad 2: +36V -> GND
- U1 pad 11: Net-(U1-Pad11) -> +3V3
- U1 pad 14: Net-(U1-Pad14) -> (no net)
- U1 pad 15: GND -> Net-(J6-Pad1)
- U1 pad 16: GND -> Net-(J6-Pad2)
- U1 pad 17: GND -> Net-(J6-Pad3)
- U1 pad 19: Net-(U1-Pad19) -> (no net)
- U1 pad 20: Net-(U1-Pad20) -> (no net)
- U1 pad 28: Net-(U1-Pad28) -> (no net)
Routing:
- net GND: track 1050.7 -> 318.2 mm
- net +3V3: track 987.9 -> 285.6 mm, vias 1 -> 0
- net +36V: track 614.5 -> 145.9 mm
- net /RPI_GPIO3: track 229.1 -> 9.58 mm
- net /RPI_GPIO2: track 232.2 -> 13.7 mm
- net /M10_3: track 132.3 -> 0.00 mm
- net /M10_2: track 123.7 -> 0.00 mm
- net /M10_1: track 118.4 -> 0.00 mm
- net /M9_3: track 115.6 -> 0.00 mm
- net /M9_1: track 104.8 -> 0.00 mm, vias 1 -> 0
- net /M9_2: track 102.9 -> 0.00 mm
- net /M20_1: track 98.4 -> 0.00 mm
- net /M8_3: track 93.3 -> 0.00 mm
- net /M20_3: track 92.2 -> 0.00 mm
- net /M20_2: track 90.3 -> 0.00 mm
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Other:
- board size 270.5 x 115.6 mm -> 141 x 57.2 mm
- board text added: "1.1"
- board text added: "100uF 50V"
- board text added: "28/03/2020"
- board text added: "3.3V"
- board text added: "3.3V input"
- board text added: "36V input"
- board text added: "Choose address"
- board text added: "GND input"
- board text added: "SolarOSE v1.1"
- board text removed: "1A"
- board text removed: "1B"
- board text removed: "2A"
- board text removed: "2B"
- board text removed: "36V"
- board text removed: "3V3"
- board text removed: "GPIO2"
- board text removed: "GPIO3"
- board text removed: "SolarOSE v1.0"
